File: dds-sweeper-board/dds-sweeper-board.kicad_pcb (KiCad board)
At the start: 2 copper layers, 56 x 65 mm, 10 parts, among them J1 REF CLK, J2 3V3, J3 1V8, J4 Headers for AD9959 Eval Board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, J5 Trigger In, SW1 Pico Power Switch, U1 Pico, U3 5V->1V8 Linear Regulator

Commit message: Minor tweaks to the breakout board.
Adds filter capacitors to the 3.3V line.

Tweaks some KiCAD options to suppress errors and warnings.
Added labels to lines going to the AD9959
Parts:
- added C3: 1uF, Capacitor_SMD:C_0805_2012Metric_Pad1.18x1.45mm_HandSolder, F.Cu at (74.0, 47.4)
- added C4: 0.1uF, Capacitor_SMD:C_0805_2012Metric_Pad1.18x1.45mm_HandSolder, F.Cu at (76.1, 49.6)
Connections:
- net Net-(J1-In) renamed /PIN_CLOCK
- net Net-(J4-Pin_1) renamed /PIN_MOSI
- net Net-(J4-Pin_11) renamed /PIN_SCK
- net Net-(J4-Pin_12) renamed /PIN_RESET
- net Net-(J4-Pin_14) renamed /PIN_SYNC
- net Net-(J4-Pin_15) renamed /PIN_MISO
- net Net-(J4-Pin_5) renamed /P0
- net Net-(J4-Pin_6) renamed /P1
- net Net-(J4-Pin_7) renamed /P2
- net Net-(J4-Pin_8) renamed /P3
- net Net-(J4-Pin_9) renamed /PIN_UPDATE
- net Net-(J5-In) renamed /TRIG_IN
- U1 pad 33: unconnected-(U1-AGND-Pad33) -> GND
