File: dds-sweeper-board/dds-sweeper-board.kicad_sch (KiCad schematic)
At the start: 10 parts, among them J1 REF CLK, J2 3V3, J3 1V8, J4 Headers for AD9959 Eval Board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, J5 Trigger In, SW1 Pico Power Switch, U1 Pico, U3 5V->1V8 Linear Regulator

Commit message: Minor tweaks to the breakout board.
Adds filter capacitors to the 3.3V line.

Tweaks some KiCAD options to suppress errors and warnings.
Added labels to lines going to the AD9959
Parts:
- added C3: 1uF, Capacitor_SMD:C_0805_2012Metric_Pad1.18x1.45mm_HandSolder, symbol Device:C
- added C4: 0.1uF, Capacitor_SMD:C_0805_2012Metric_Pad1.18x1.45mm_HandSolder, symbol Device:C
Connections:
- net 3V3: now also C3.2, C4.2
- net GND: now also U1.33 (AGND), C3.1, C4.1
- net TRIG_IN: now reaches J5.1 (In), U1.11 (GPIO8)
- net PIN_RESET: now reaches J4.12 (Pin_12), U1.12 (GPIO9)
- net PIN_SYNC: now reaches J4.14 (Pin_14), U1.14 (GPIO10)
- net PIN_MISO: now reaches J4.15 (Pin_15), U1.16 (GPIO12)
- net PIN_SCK: now reaches J4.11 (Pin_11), U1.19 (GPIO14)
- net PIN_MOSI: now reaches J4.1 (Pin_1), U1.20 (GPIO15)
- net P3: now reaches J4.8 (Pin_8), U1.21 (GPIO16)
- net P2: now reaches J4.7 (Pin_7), U1.22 (GPIO17)
- net P1: now reaches J4.6 (Pin_6), U1.24 (GPIO18)
- net P0: now reaches J4.5 (Pin_5), U1.25 (GPIO19)
- net PIN_CLOCK: now reaches J1.1 (In), U1.27 (GPIO21)
- net PIN_UPDATE: now reaches J4.9 (Pin_9), U1.29 (GPIO22)
- no-connect marks 33 -> 23
